Commit message: Add the robotiq 85 gripper to the ur3e model

File: src/orendes_description/urdf/orendes_85_gripper.urdf.xacro (robot description, xacro)
@@ -31,5 +31,5 @@
             <child link="${prefix}orendes_85_left_finger_tip_link"/>
             <axis xyz="0 0 1"/>
-            <origin rpy="${pi} 0.0 0.0" xyz="0.05490451627 0.03060114443 0.0"/>
+            <origin rpy="${pi} 0.0 0.0" xyz="0.05490451627 0.03060114443 0.1"/>
             <limit lower="0.0" upper="0.804" velocity="2.0" effort="1000"/>
         </joint>

Commit message: Adjust tips to the main link

File: src/orendes_description/urdf/orendes_85_gripper.urdf.xacro (robot description, xacro)
@@ -23,21 +23,23 @@
                 <origin xyz="0.0 0.0 0.0" />
                 <inertia ixx="0.000380" ixy="0.000000" ixz="0.000000"
-                        iyx="0.000000" iyy="0.001110" iyz="0.000000"
-                        izx="0.000000" izy="0.000000" izz="0.001171" />
+                         iyx="0.000000" iyy="0.001110" iyz="0.000000"
+                         izx="0.000000" izy="0.000000" izz="0.001171" />
             </inertial>
         </link>
+        <!--left tip -->
         <joint name="${prefix}orendes_85_left_finger_tip_joint" type="revolute">
             <parent link="${prefix}orendes_85_base_link"/>
             <child link="${prefix}orendes_85_left_finger_tip_link"/>
             <axis xyz="0 0 1"/>
-            <origin rpy="${pi} 0.0 0.0" xyz="0.05490451627 0.03060114443 0.1"/>
-            <limit lower="0.0" upper="0.804" velocity="2.0" effort="1000"/>
+            <origin rpy="0.0001 0.0 0.0" xyz="-0.0199 0.008 0.045"/>
+            <limit lower="-3.14" upper="3.14" velocity="100.0" effort="0.1"/>
         </joint>
+        <!--right tip-->
         <joint name="${prefix}orendes_85_right_finger_tip_joint" type="continuous">
             <parent link="${prefix}orendes_85_base_link"/>
             <child link="${prefix}orendes_85_right_finger_tip_link"/>
             <axis xyz="0 0 1"/>
-            <origin rpy="0.0 0.0 0.0" xyz="0.05490451627 -0.03060114443 0.0"/>
-            <limit lower="-3.14" upper="3.14" velocity="100.0" effort="1000"/>
+            <origin rpy="0.0 0.0 0.0" xyz="0.2545451627 -0.03180114443 0.0629"/>
+            <limit lower="-3.14" upper="3.14" velocity="100.0" effort="0.1"/>
             <mimic joint="${prefix}orendes_85_left_finger_tip_joint"/>
         </joint>

Commit message: Attach the gripper to the robot

File: src/orendes_description/urdf/orendes_85_gripper.urdf.xacro (robot description, xacro)
@@ -27,5 +27,4 @@
             </inertial>
         </link>
-        <!--left tip -->
         <joint name="${prefix}orendes_85_left_finger_tip_joint" type="revolute">
             <parent link="${prefix}orendes_85_base_link"/>
@@ -35,5 +34,4 @@
             <limit lower="-3.14" upper="3.14" velocity="100.0" effort="0.1"/>
         </joint>
-        <!--right tip-->
         <joint name="${prefix}orendes_85_right_finger_tip_joint" type="continuous">
             <parent link="${prefix}orendes_85_base_link"/>

File: src/ur3e_description/urdf/orendes_85_eef.xacro (robot description, xacro)
@@ -5,5 +5,5 @@
     <!-- Call the gripper macro with correct parameters -->
     <xacro:orendes_85_gripper prefix="" parent="tool0">
-        <origin xyz="0 0 0" rpy="0 0 -1.57">
+        <origin xyz="0.08 0 0" rpy="-1.5708 0 -1.5708"/>
     </xacro:orendes_85_gripper>
 </robot>

Commit message: Fix values

File: src/orendes_description/urdf/orendes_85_gripper.urdf.xacro (robot description, xacro)
@@ -27,9 +27,9 @@
             </inertial>
         </link>
-        <joint name="${prefix}orendes_85_left_finger_tip_joint" type="revolute">
+        <joint name="${prefix}orendes_85_left_finger_tip_joint" type="continuous">
             <parent link="${prefix}orendes_85_base_link"/>
             <child link="${prefix}orendes_85_left_finger_tip_link"/>
             <axis xyz="0 0 1"/>
-            <origin rpy="0.0001 0.0 0.0" xyz="-0.0199 0.008 0.045"/>
+            <origin rpy="0.0 0.0 0.0" xyz="-0.0199 0.008 0.045"/>
             <limit lower="-3.14" upper="3.14" velocity="100.0" effort="0.1"/>
         </joint>
@@ -40,5 +40,5 @@
             <origin rpy="0.0 0.0 0.0" xyz="0.2545451627 -0.03180114443 0.0629"/>
             <limit lower="-3.14" upper="3.14" velocity="100.0" effort="0.1"/>
-            <mimic joint="${prefix}orendes_85_left_finger_tip_joint"/>
+            <mimic joint="${prefix}orendes_85_left_finger_tip_joint" multiplier="-1"/>
         </joint>
         <link name="${prefix}orendes_85_left_finger_tip_link">

Commit message: Change to prismatic type of movable tips

File: src/orendes_description/urdf/orendes_85_gripper.urdf.xacro (robot description, xacro)
@@ -27,19 +27,23 @@
             </inertial>
         </link>
-        <joint name="${prefix}orendes_85_left_finger_tip_joint" type="continuous">
+        <!-- Left Finger Joint -->
+        <joint name="${prefix}orendes_85_left_finger_tip_joint" type="prismatic">
             <parent link="${prefix}orendes_85_base_link"/>
             <child link="${prefix}orendes_85_left_finger_tip_link"/>
-            <axis xyz="0 0 1"/>
+            <axis xyz="1 0 0"/>
             <origin rpy="0.0 0.0 0.0" xyz="-0.0199 0.008 0.045"/>
-            <limit lower="-3.14" upper="3.14" velocity="100.0" effort="0.1"/>
+            <limit lower="0" upper="-0.0036" velocity="0.05" effort="1000"/>
         </joint>
-        <joint name="${prefix}orendes_85_right_finger_tip_joint" type="continuous">
+        <!-- Right Finger Joint -->
+        <joint name="${prefix}orendes_85_right_finger_tip_joint" type="prismatic">
             <parent link="${prefix}orendes_85_base_link"/>
             <child link="${prefix}orendes_85_right_finger_tip_link"/>
-            <axis xyz="0 0 1"/>
+            <axis xyz="1 0 0"/>
             <origin rpy="0.0 0.0 0.0" xyz="0.2545451627 -0.03180114443 0.0629"/>
-            <limit lower="-3.14" upper="3.14" velocity="100.0" effort="0.1"/>
+            <limit lower="0" upper="-0.0036" velocity="0.05" effort="1000"/>
+            <!-- Mimic the left finger joint with inverse movement -->
             <mimic joint="${prefix}orendes_85_left_finger_tip_joint" multiplier="-1"/>
         </joint>
+        <!-- Left Finger Link -->
         <link name="${prefix}orendes_85_left_finger_tip_link">
             <visual>
@@ -56,9 +60,10 @@
                 <mass value="0.018491" />
                 <origin xyz="0.0 0.0 0.0" />
-                <inertia ixx="0.000009" ixy="-0.000001" ixz="0.000000"
-                         iyx="-0.000001" iyy="0.000001" iyz="0.000000"
-                         izx="0.000000" izy="0.000000" izz="0.000010" />
+                <inertia ixx="0.000002" ixy="0.000000" ixz="0.000000"
+                         iyx="0.000000" iyy="0.000005" iyz="0.000000"
+                         izx="0.000000" izy="0.000000" izz="0.000006" />
             </inertial>
         </link>
+        <!-- Right Finger Link -->
         <link name="${prefix}orendes_85_right_finger_tip_link">
             <visual>
@@ -75,7 +80,7 @@
                 <mass value="0.018491" />
                 <origin xyz="0.0 0.0 0.0" />
-                <inertia ixx="0.000009" ixy="-0.000001" ixz="0.000000"
-                         iyx="-0.000001" iyy="0.000001" iyz="0.000000"
-                         izx="0.000000" izy="0.000000" izz="0.000010" />
+                <inertia ixx="0.000002" ixy="0.000000" ixz="0.000000"
+                         iyx="0.000000" iyy="0.000005" iyz="0.000000"
+                         izx="0.000000" izy="0.000000" izz="0.000006" />
             </inertial>
         </link>
