Commit message: Update gripper

File: src/custom_robot_description/urdf/custom_gripper.xacro (robot description, xacro)
@@ -2,6 +2,7 @@
 <robot xmlns:xacro="http://www.ros.org.wiki.xacro">
     <xacro:include filename="$(find custom_robot_description)/urdf/link_joint.xacro"/>
-    <!-- xacro:macro for gripper -->
+    <!-- macro for the custom_gripper -->
     <xacro:macro name="custom_gripper" params="parent origin_xyz">
+        <!-- gripper_connector -->
         <xacro:cobot_link_cylinder name="gripper_connector"
             origin_xyz="0 0 0.015"
@@ -9,10 +10,47 @@
             radius="0.04"
             length="0.03"/>
-        <joint name="{parent}__gripper_connector"
-            type="fixed">
+        <!-- connect gripper_connector to the parent -->
+        <joint name="{parent}__gripper_connector" type="fixed">
             <parent link="${parent}"/>
             <child link="gripper_connector"/>
             <origin xyz="${origin_xyz}" rpy="0 0 0"/>
         </joint>
+        <!-- finger_support -->
+        <xacro:cobot_link_box name="finger_support"
+            origin_xyz="0 0.005 0.005"
+            origin_rpy="0 0 0"
+            size="0.120 0.01 0.01"/>
+        <!-- connect gripper_connector to finger_support -->
+        <joint name="finger_support__gripper_connector" type="fixed">
+            <parent link="gripper_connector"/>
+            <child link="finger_support"/>
+            <origin xyz="0 0 0.03" rpy="0 0 0"/>
+        </joint>
+        <!-- finger_right & finger_left -->
+        <xacro:cobot_link_box name="finger_right"
+            origin_xyz="0 0 0.04"
+            origin_rpy="0 0 0"
+            size="0.01 0.01 0.08"/>
+        <xacro:cobot_link_box name="finger_left"
+            origin_xyz="0 0 0.04"
+            origin_rpy="0 0 0"
+            size="0.01 0.01 0.08"/>
+        <!-- connect finger_right and finger_left to finger_support -->
+        <joint name="finger_right_joint" type="prismatic">
+            <parent link="finger_support"/>
+            <child link="finger_right"/>
+            <axis xyz="1 0 0"/>
+            <limit lower="0" upper="0.044" effort="200" velocity="0.5"/>
+            <origin xyz="-0.05 0 0.01" rpy="0 0 0"/>
+            <dynamics damping="1" friction="2"/>
+        </joint>
+        <joint name="finger_left_joint" type="prismatic">
+            <parent link="finger_support"/>
+            <child link="finger_left"/>
+            <axis xyz="1 0 0"/>
+            <limit lower="-0.044" upper="0" effort="200" velocity="0.5"/>
+            <origin xyz="0.05 0 0.01" rpy="0 0 0"/>
+            <dynamics damping="1" friction="2"/>
+        </joint>
     </xacro:macro>
 </robot>

File: src/custom_robot_description/urdf/link_joint.xacro (robot description, xacro)
@@ -1,5 +1,5 @@
 <?xml version = "1.0"?>
 <robot xmlns:xacro="http://www.ros.org.wiki.xacro">
-    <!-- xacro:macro for links -->
+    <!-- macro for the links -->
     <xacro:macro name="cobot_link_cylinder" params="name origin_xyz origin_rpy radius length">
         <link name="${name}">
@@ -18,5 +18,22 @@
         </link>
     </xacro:macro>
-    <!-- xacro:macro for joints -->
+    <!-- macro for finger_support -->
+    <xacro:macro name="cobot_link_box" params="name origin_xyz origin_rpy size">
+        <link name="${name}">
+            <visual>
+                <geometry>
+                    <box size="${size}"/>
+                </geometry>
+                <origin xyz="${origin_xyz}" rpy="${origin_rpy}"/>
+            </visual>
+            <collision>
+                <geometry>
+                    <box size="${size}"/>
+                </geometry>
+                <origin xyz="${origin_xyz}" rpy="${origin_rpy}"/>
+            </collision>
+        </link>
+    </xacro:macro>
+    <!-- macro for the joints -->
     <xacro:macro name="cobot_joint" params="name type parent child axis limit_l limit_u limit_v limit_e origin_xyz origin_rpy">
         <joint name="${name}" type="${type}">

Commit message: Add inertia values

File: src/custom_robot_description/urdf/custom_gripper.xacro (robot description, xacro)
@@ -1,2 +1,3 @@
+<!-- Inetia is calculated with: https://en.wikipedia.org/wiki/List_of_moments_of_inertia -->
 <?xml version = "1.0"?>
 <robot xmlns:xacro="http://www.ros.org.wiki.xacro">
@@ -6,8 +7,15 @@
         <!-- gripper_connector -->
         <xacro:cobot_link_cylinder name="gripper_connector"
-            origin_xyz="0 0 0.015"
-            origin_rpy="0 0 0"
+            origin_xyz="0.0 0.0 0.015"
+            origin_rpy="0.0 0.0 0.0"
             radius="0.04"
-            length="0.03"/>
+            length="0.03"
+            mass="0.5"
+            i_xx="0.002375"
+            i_xy="0.0"
+            i_xz="0.0"
+            i_yy="0.002375"
+            i_yz="0.0"
+            i_zz="0.00006666666667"/>
         <!-- connect gripper_connector to the parent -->
         <joint name="{parent}__gripper_connector" type="fixed">
@@ -18,7 +26,14 @@
         <!-- finger_support -->
         <xacro:cobot_link_box name="finger_support"
-            origin_xyz="0 0.005 0.005"
-            origin_rpy="0 0 0"
-            size="0.120 0.01 0.01"/>
+            origin_xyz="0.0 0.005 0.005"
+            origin_rpy="0.0 0.0 0.0"
+            size="0.120 0.01 0.01"
+            mass="0.25"
+            i_xx="0.0003"
+            i_xy="0.0"
+            i_xz="0.0"
+            i_yy="0.0"
+            i_yz="0.0"
+            i_zz="0.0003"/>
         <!-- connect gripper_connector to finger_support -->
         <joint name="finger_support__gripper_connector" type="fixed">
@@ -31,9 +46,23 @@
             origin_xyz="0 0 0.04"
             origin_rpy="0 0 0"
-            size="0.01 0.01 0.08"/>
+            size="0.01 0.01 0.08"
+            mass="0.2"
+            i_xx="0.00042667"
+            i_xy="0.0"
+            i_xz="0.0"
+            i_yy="0.0"
+            i_yz="0.0"
+            i_zz="0.00042667"/>
         <xacro:cobot_link_box name="finger_left"
             origin_xyz="0 0 0.04"
             origin_rpy="0 0 0"
-            size="0.01 0.01 0.08"/>
+            size="0.01 0.01 0.08"
+            mass="0.2"
+            i_xx="0.00042667"
+            i_xy="0.0"
+            i_xz="0.0"
+            i_yy="0.0"
+            i_yz="0.0"
+            i_zz="0.00042667"/>
         <!-- connect finger_right and finger_left to finger_support -->
         <joint name="finger_right_joint" type="prismatic">

File: src/custom_robot_description/urdf/link_joint.xacro (robot description, xacro)
@@ -1,7 +1,12 @@
 <?xml version = "1.0"?>
 <robot xmlns:xacro="http://www.ros.org.wiki.xacro">
-    <!-- macro for the links -->
-    <xacro:macro name="cobot_link_cylinder" params="name origin_xyz origin_rpy radius length">
+    <!-- macro for the links (cylinders) -->
+    <xacro:macro name="cobot_link_cylinder" params="name origin_xyz origin_rpy radius length mass i_xx i_xy i_xz i_yy i_yz i_zz">
         <link name="${name}">
+            <inertial>
+                <origin xyz="${origin_xyz}" rpy="${origin_rpy}"/>
+                <mass value="${mass}"/>
+                <inertia ixx="${i_xx}" ixy="${i_xy}" ixz="${i_xz}"  iyy="${i_yy}" iyz="${i_yz}" izz="${i_zz}"/>
+            </inertial>
             <visual>
                 <geometry>
@@ -19,6 +24,11 @@
     </xacro:macro>
     <!-- macro for finger_support -->
-    <xacro:macro name="cobot_link_box" params="name origin_xyz origin_rpy size">
+    <xacro:macro name="cobot_link_box" params="name origin_xyz origin_rpy size mass i_xx i_xy i_xz i_yy i_yz i_zz">
         <link name="${name}">
+            <inertial>
+                <origin xyz="${origin_xyz}" rpy="${origin_rpy}"/>
+                <mass value="${mass}"/>
+                <inertia ixx="${i_xx}" ixy="${i_xy}" ixz="${i_xz}"  iyy="${i_yy}" iyz="${i_yz}" izz="${i_zz}"/>
+            </inertial>
             <visual>
                 <geometry>
@@ -35,5 +45,5 @@
         </link>
     </xacro:macro>
-    <!-- macro for the joints -->
+    <!-- macro for the joints (connections) -->
     <xacro:macro name="cobot_joint" params="name type parent child axis limit_l limit_u limit_v limit_e origin_xyz origin_rpy">
         <joint name="${name}" type="${type}">
